Commit message: feat(slam): add Gazebo mapping and localization

File: src/inspection_robot_description/urdf/base.xacro (robot description, xacro)
@@ -3,5 +3,5 @@
   <xacro:macro
     name="base"
-    params="length width height mass base_link_z">
+    params="length width height mass base_link_z chassis_x chassis_z com_x com_z">
     <!--
       base_footprint 是地面投影坐标系，没有 visual、collision 和质量。
@@ -10,29 +10,41 @@
     <!-- 实际底盘刚体 -->
     <link name="base_link">
-      <visual>
-        <geometry>
-          <box size="${length} ${width} ${height}"/>
-        </geometry>
-        <material name="base_blue">
-          <color rgba="0.2 0.45 0.8 1.0"/>
-        </material>
-      </visual>
-      <collision>
-        <geometry>
-          <box size="${length} ${width} ${height}"/>
-        </geometry>
-      </collision>
-      <!-- 长方体绕自身质心的惯性矩阵 -->
-      <inertial>
-        <mass value="${mass}"/>
-        <inertia
-          ixx="${mass * (width * width + height * height) / 12.0}"
-          ixy="0.0"
-          ixz="0.0"
-          iyy="${mass * (length * length + height * height) / 12.0}"
-          iyz="0.0"
-          izz="${mass * (length * length + width * width) / 12.0}"/>
-      </inertial>
-    </link>
+    <visual>
+      <origin
+        xyz="${chassis_x} 0 ${chassis_z}"
+        rpy="0 0 0"/>
+      <geometry>
+        <box size="${length} ${width} ${height}"/>
+      </geometry>
+      <material name="base_blue">
+        <color rgba="0.2 0.45 0.8 1.0"/>
+      </material>
+    </visual>
+    <collision>
+      <origin
+        xyz="${chassis_x} 0 ${chassis_z}"
+        rpy="0 0 0"/>
+      <geometry>
+        <box size="${length} ${width} ${height}"/>
+      </geometry>
+    </collision>
+    <inertial>
+      <!--
+            惯性参考点设在简化后的质心。
+           当前仍用长方体惯量作为第一版物理近似。
+      -->
+      <origin
+        xyz="${com_x} 0 ${com_z}"
+        rpy="0 0 0"/>
+      <mass value="${mass}"/>
+      <inertia
+        ixx="${mass * (width * width + height * height) / 12.0}"
+        ixy="0.0"
+        ixz="0.0"
+        iyy="${mass * (length * length + height * height) / 12.0}"
+        iyz="0.0"
+        izz="${mass * (length * length + width * width) / 12.0}"/>
+    </inertial>
+  </link>
     <!-- base_link 位于地面上方 -->
     <joint name="base_footprint_joint" type="fixed">

File: src/inspection_robot_description/urdf/inspection_robot.urdf.xacro (robot description, xacro)
@@ -3,4 +3,9 @@
   name="inspection_robot"
   xmlns:xacro="http://www.ros.org/wiki/xacro">
+  <!-- 选择 ros2_control 后端：
+       false = Mock GenericSystem
+       true  = GazeboSystem -->
+  <xacro:arg name="use_gazebo" default="false"/>
+  <xacro:arg name="controllers_file" default=""/>
   <!-- 参数表 -->
   <xacro:include filename="robot_properties.xacro"/>
@@ -8,4 +13,5 @@
   <xacro:include filename="base.xacro"/>
   <xacro:include filename="wheel.xacro"/>
+  <xacro:include filename="caster.xacro"/>
   <xacro:include filename="sensors/laser.xacro"/>
   <xacro:include filename="sensors/imu.xacro"/>
@@ -18,5 +24,9 @@
     height="${base_height}"
     mass="${base_mass}"
-    base_link_z="${base_link_z}"/>
+    base_link_z="${base_link_z}"
+    chassis_x="${chassis_x}"
+    chassis_z="${chassis_z}"
+    com_x="${base_com_x}"
+    com_z="${base_com_z}"/>
   <!-- 创建左轮：ROS 坐标系中 Y 正方向为左侧 -->
   <xacro:wheel
@@ -37,9 +47,17 @@
     y="${-wheel_separation / 2.0}"
     z="${wheel_z}"/>
+  <!-- 后部万向支撑球 -->
+  <xacro:caster
+    radius="${caster_radius}"
+    mass="${caster_mass}"
+    x="${caster_x}"
+    y="${caster_y}"
+    z="${caster_z}"/>
   <!-- 激光雷达 -->
   <xacro:laser
     x="${laser_x}"
     y="${laser_y}"
-    z="${laser_z}"/>
+    z="${laser_z}"
+    use_gazebo="$(arg use_gazebo)"/>
   <!-- IMU -->
   <xacro:imu
@@ -48,4 +66,6 @@
     z="${imu_z}"/>
   <!-- ros2_control -->
-  <xacro:inspection_robot_ros2_control/>
+  <xacro:inspection_robot_ros2_control
+    use_gazebo="$(arg use_gazebo)"
+    controllers_file="$(arg controllers_file)"/>
 </robot>

File: src/inspection_robot_description/urdf/robot_properties.xacro (robot description, xacro)
@@ -1,32 +1,57 @@
 <?xml version="1.0"?>
 <robot xmlns:xacro="http://www.ros.org/wiki/xacro">
-  <!-- 底盘尺寸，单位均为 SI：米、千克 -->
+  <!-- 底盘外形尺寸 -->
   <xacro:property name="base_length" value="0.32"/>
   <xacro:property name="base_width"  value="0.24"/>
   <xacro:property name="base_height" value="0.10"/>
   <xacro:property name="base_mass"   value="4.0"/>
-  <!-- base_link 原点距离地面的高度 -->
-  <xacro:property name="base_link_z" value="0.08"/>
-  <!-- 左右驱动轮参数 -->
+  <!--
+    V2 坐标定义：
+    base_link 位于左右驱动轮轴线中点，
+        高度等于驱动轮半径。
+  -->
+  <xacro:property name="base_link_z" value="0.05"/>
+  <!--
+        底盘几何体相对于 base_link 的位置。
+        底盘向后偏 4 cm；
+        底部离地 3 cm，因此几何中心 z=0.03。
+  -->
+  <xacro:property name="chassis_x" value="-0.04"/>
+  <xacro:property name="chassis_z" value="0.03"/>
+  <!--
+        简化的整机质心位置。
+        重部件假设低位、略微偏后。
+  -->
+  <xacro:property name="base_com_x" value="-0.05"/>
+  <xacro:property name="base_com_z" value="0.00"/>
+  <!-- 左右驱动轮 -->
   <xacro:property name="wheel_radius"     value="0.05"/>
   <xacro:property name="wheel_width"      value="0.02"/>
   <xacro:property name="wheel_mass"       value="0.30"/>
   <xacro:property name="wheel_separation" value="0.28"/>
-  <!-- 轮子位于底盘中心的前后位置 -->
+  <!-- 驱动轮轴线就是 base_link 的 X=0 -->
   <xacro:property name="wheel_x" value="0.0"/>
   <!--
-    轮子中心离地高度为 wheel_radius。
-    下面计算的是轮子相对 base_link 的 Z 坐标。
+    base_link 高度已经等于轮半径，
+        所以轮心与 base_link 位于同一高度。
   -->
   <xacro:property
     name="wheel_z"
     value="${wheel_radius - base_link_z}"/>
-      <!-- 2D 激光雷达相对于 base_link 的安装位置 -->
-  <xacro:property name="laser_x" value="0.10"/>
+  <!-- 后部支撑球 -->
+  <xacro:property name="caster_radius" value="0.025"/>
+  <xacro:property name="caster_mass"   value="0.05"/>
+  <xacro:property name="caster_x" value="-0.13"/>
+  <xacro:property name="caster_y" value="0.0"/>
+  <xacro:property
+    name="caster_z"
+    value="${caster_radius - base_link_z}"/>
+  <!-- 2D 激光雷达相对于 base_link 的安装位置 -->
+  <xacro:property name="laser_x" value="0.05"/>
   <xacro:property name="laser_y" value="0.0"/>
-  <xacro:property name="laser_z" value="0.15"/>
+  <xacro:property name="laser_z" value="0.10"/>
   <!-- IMU 相对于 base_link 的安装位置 -->
   <xacro:property name="imu_x" value="0.0"/>
   <xacro:property name="imu_y" value="0.0"/>
-  <xacro:property name="imu_z" value="0.06"/>
+  <xacro:property name="imu_z" value="0.03"/>
 </robot>

File: src/inspection_robot_description/urdf/ros2_control.xacro (robot description, xacro)
@@ -1,9 +1,18 @@
 <?xml version="1.0"?>
 <robot xmlns:xacro="http://www.ros.org/wiki/xacro">
-  <xacro:macro name="inspection_robot_ros2_control">
+  <xacro:macro
+  name="inspection_robot_ros2_control"
+  params="use_gazebo controllers_file">
     <ros2_control name="InspectionRobotSystem" type="system">
       <hardware>
-        <plugin>mock_components/GenericSystem</plugin>
-        <param name="calculate_dynamics">true</param>
+        <!-- Gazebo 仿真 -->
+        <xacro:if value="${use_gazebo}">
+          <plugin>gazebo_ros2_control/GazeboSystem</plugin>
+        </xacro:if>
+        <!-- 默认 Mock Hardware -->
+        <xacro:unless value="${use_gazebo}">
+          <plugin>mock_components/GenericSystem</plugin>
+          <param name="calculate_dynamics">true</param>
+        </xacro:unless>
       </hardware>
       <joint name="left_wheel_joint">
@@ -22,4 +31,15 @@
       </joint>
     </ros2_control>
+    <xacro:if value="${use_gazebo}">
+      <gazebo>
+        <plugin
+          filename="libgazebo_ros2_control.so"
+          name="gazebo_ros2_control">
+          <robot_param>robot_description</robot_param>
+          <robot_param_node>robot_state_publisher</robot_param_node>
+          <parameters>${controllers_file}</parameters>
+        </plugin>
+      </gazebo>
+    </xacro:if>
   </xacro:macro>
 </robot>

File: src/inspection_robot_description/urdf/sensors/laser.xacro (robot description, xacro)
@@ -1,5 +1,5 @@
 <?xml version="1.0"?>
 <robot xmlns:xacro="http://www.ros.org/wiki/xacro">
-  <xacro:macro name="laser" params="x y z">
+  <xacro:macro name="laser" params="x y z use_gazebo">
     <link name="laser_link">
       <visual>
@@ -24,4 +24,42 @@
         rpy="0 0 0"/>
     </joint>
+    <xacro:if value="${use_gazebo}">
+      <gazebo reference="laser_link">
+        <sensor name="laser_sensor" type="ray">
+          <always_on>true</always_on>
+          <visualize>true</visualize>
+          <update_rate>10.0</update_rate>
+          <ray>
+            <scan>
+              <horizontal>
+                <samples>360</samples>
+                <resolution>1</resolution>
+                <min_angle>-3.14159265</min_angle>
+                <max_angle>3.14159265</max_angle>
+              </horizontal>
+            </scan>
+            <range>
+              <min>0.12</min>
+              <max>8.0</max>
+              <resolution>0.01</resolution>
+            </range>
+            <noise>
+              <type>gaussian</type>
+              <mean>0.0</mean>
+              <stddev>0.01</stddev>
+            </noise>
+          </ray>
+          <plugin
+            name="gazebo_ros_ray_sensor"
+            filename="libgazebo_ros_ray_sensor.so">
+            <ros>
+              <remapping>~/out:=/scan</remapping>
+            </ros>
+            <output_type>sensor_msgs/LaserScan</output_type>
+            <frame_name>laser_link</frame_name>
+          </plugin>
+        </sensor>
+      </gazebo>
+    </xacro:if>
   </xacro:macro>
 </robot>
